File: examples/aquila_gps.kicad_pcb (KiCad board)
At the start: 2 copper layers, 399 x 120 mm, 0 parts

Commit message: implemented directions for components
Other:
- board size 399 x 120 mm -> 399 x 160 mm
Changed lines of the file:
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@@
     (gr_poly
     (pts
-      (xy 245.34383269322396 150.451953125)
-      (xy 245.34383269322396 149.203515625)
-      (xy 308.9490823764759 149.203515625)
-      (xy 308.9490823764759 140)
-      (xy 310.54205112647594 140)
-      (xy 310.54205112647594 140.451953125)
-      (xy 345.0893994446999 140.451953125)
-      (xy 345.0893994446999 139.203515625)
-      (xy 358.82186575221385 139.203515625)
-      (xy 358.82186575221385 130)
-      (xy 360.4148345022139 130)
-      (xy 360.4148345022139 139.10925688501632)
-      (xy 358.72760701223024 140.796484375)
-      (xy 345.0893994446999 140.796484375)
-      (xy 345.0893994446999 139.548046875)
-      (xy 274.401734058252 139.548046875)
-      (xy 274.401734058252 139.203515625)
-      (xy 260.66926775073796 139.203515625)
-      (xy 260.66926775073796 130)
-      (xy 259.07629900073795 130)
-      (xy 259.07629900073795 139.10925688501632)
-      (xy 260.5750090107543 140.796484375)
-      (xy 274.401734058252 140.796484375)
-      (xy 274.401734058252 140.451953125)
-      (xy 308.9490823764759 140.451953125)
-      (xy 308.9490823764759 140)
-      (xy 310.54205112647594 140)
-      (xy 310.54205112647594 149.10925688501632)
-      (xy 308.85482363649226 150.796484375)
-      (xy 245.34383269322396 150.796484375)
-      (xy 245.34383269322396 149.548046875)
-      (xy 174.65616730677604 149.548046875)
-      (xy 174.65616730677604 149.203515625)
-      (xy 111.05091762352407 149.203515625)
-      (xy 111.05091762352407 140)
-      (xy 111.05091762352407 140)
-      (xy 111.05091762352407 140.451953125)
-      (xy 145.59826594174802 140.451953125)
-      (xy 145.59826594174802 139.203515625)
-      (xy 159.33073224926204 139.203515625)
-      (xy 159.33073224926204 130)
-      (xy 160.92370099926202 130)
-      (xy 160.92370099926202 139.10925688501632)
-      (xy 159.23647350927837 140.796484375)
-      (xy 145.59826594174802 140.796484375)
-      (xy 145.59826594174802 139.548046875)
-      (xy 74.9106005553001 139.548046875)
-      (xy 74.9106005553001 139.203515625)
-      (xy 61.17813424778612 139.203515625)
-      (xy 61.17813424778612 130)
-      (xy 59.58516549778611 130)
-      (xy 59.58516549778611 139.10925688501632)
-      (xy 61.083875507802446 140.796484375)
-      (xy 74.9106005553001 140.796484375)
-      (xy 74.9106005553001 140.451953125)
-      (xy 109.45794887352406 140.451953125)
-      (xy 109.45794887352406 140)
-      (xy 109.45794887352406 140)
-      (xy 109.45794887352406 149.10925688501632)
-      (xy 110.9566588835404 150.796484375)
-      (xy 174.65616730677604 150.796484375)
-      (xy 174.65616730677604 150.451953125)
-      (xy 210 150.451953125)
-      (xy 210 150.3)
-      (xy 209.7 150)
-      (xy 210 149.7)
-      (xy 210.3 150)
-      (xy 210 150.3)
-      (xy 210 150.451953125)
+      (xy 245.34383269322396 200.451953125)
+      (xy 245.34383269322396 199.203515625)
+      (xy 308.9490823764759 199.203515625)
+      (xy 308.9490823764759 190)
+      (xy 310.54205112647594 190)
+      (xy 310.54205112647594 190.451953125)
+      (xy 345.0893994446999 190.451953125)
+      (xy 345.0893994446999 189.203515625)
+      (xy 358.82186575221385 189.203515625)
+      (xy 358.82186575221385 180)
+      (xy 359.9411040334639 180)
+      (xy 359.9411040334639 144.36135869805292)
+      (xy 397.26451274826604 144.36135869805292)
+      (xy 397.26451274826604 80.34774264352149)
+      (xy 321.97218750616173 80.34774264352149)
+      (xy 321.97218750616173 144.36135869805292)
+      (xy 359.2955962209639 144.36135869805292)
+      (xy 359.2955962209639 180)
+      (xy 360.4148345022139 180)
+      (xy 360.4148345022139 189.10925688501632)
+      (xy 358.72760701223024 190.796484375)
+      (xy 345.0893994446999 190.796484375)
+      (xy 345.0893994446999 189.548046875)
+      (xy 274.401734058252 189.548046875)
+      (xy 274.401734058252 189.203515625)
+      (xy 260.66926775073796 189.203515625)
+      (xy 260.66926775073796 180)
+      (xy 260.195537281988 180)
+      (xy 260.195537281988 144.36135869805292)
+      (xy 297.5189459967901 144.36135869805292)
+      (xy 297.5189459967901 80.34774264352149)
+      (xy 222.22662075468583 80.34774264352149)
+      (xy 222.22662075468583 144.36135869805292)
+      (xy 259.550029469488 144.36135869805292)
+      (xy 259.550029469488 180)
+      (xy 259.07629900073795 180)
+      (xy 259.07629900073795 189.10925688501632)
+      (xy 260.76352649072163 190.796484375)
+      (xy 274.401734058252 190.796484375)
+      (xy 274.401734058252 190.451953125)
+      (xy 308.9490823764759 190.451953125)
+      (xy 308.9490823764759 190)
+      (xy 310.54205112647594 190)
+      (xy 310.54205112647594 199.10925688501632)
+      (xy 308.85482363649226 200.796484375)
+      (xy 245.34383269322396 200.796484375)
+      (xy 245.34383269322396 199.548046875)
+      (xy 174.65616730677604 199.548046875)
+      (xy 174.65616730677604 199.203515625)
+      (xy 111.05091762352407 199.203515625)
+      (xy 111.05091762352407 190)
+      (xy 111.05091762352407 190)
+      (xy 111.05091762352407 190.451953125)
+      (xy 145.59826594174802 190.451953125)
+      (xy 145.59826594174802 189.203515625)
+      (xy 159.33073224926204 189.203515625)
+      (xy 159.33073224926204 180)
+      (xy 160.44997053051202 180)
+      (xy 160.44997053051202 144.36135869805292)
+      (xy 197.77337924531417 144.36135869805292)
+      (xy 197.77337924531417 80.34774264352149)
+      (xy 122.48105400320989 80.34774264352149)
+      (xy 122.48105400320989 144.36135869805292)
+      (xy 159.80446271801202 144.36135869805292)
+      (xy 159.80446271801202 180)
+      (xy 160.92370099926202 180)
+      (xy 160.92370099926202 189.10925688501632)
+      (xy 159.23647350927837 190.796484375)
+      (xy 145.59826594174802 190.796484375)
+      (xy 145.59826594174802 189.548046875)
+      (xy 74.9106005553001 189.548046875)
+      (xy 74.9106005553001 189.203515625)
+      (xy 61.17813424778612 189.203515625)
+      (xy 61.17813424778612 180)
+      (xy 60.70440377903611 180)
+      (xy 60.70440377903611 144.36135869805292)
+      (xy 98.02781249383824 144.36135869805292)
+      (xy 98.02781249383824 80.34774264352149)
+      (xy 22.735487251733986 80.34774264352149)
+      (xy 22.735487251733986 144.36135869805292)
+      (xy 60.05889596653611 144.36135869805292)
+      (xy 60.05889596653611 180)
+      (xy 59.58516549778611 180)
+      (xy 59.58516549778611 189.10925688501632)
+      (xy 61.27239298776979 190.796484375)
+      (xy 74.9106005553001 190.796484375)
+      (xy 74.9106005553001 190.451953125)
+      (xy 109.45794887352406 190.451953125)
+      (xy 109.45794887352406 190)
+      (xy 109.45794887352406 190)
+      (xy 109.45794887352406 199.10925688501632)
+      (xy 111.14517636350774 200.796484375)
+      (xy 174.65616730677604 200.796484375)
+      (xy 174.65616730677604 200.451953125)
+      (xy 210 200.451953125)
+      (xy 210 200.3)
+      (xy 209.7 200)
+      (xy 210 199.7)
+      (xy 210.3 200)
+      (xy 210 200.3)
+      (xy 210 200.451953125)
     )
-  (layer "F.Cu") (width 0) (fill solid))(gr_rect (start 10.508866497048132 50) (end 409.49113350295187 170) (layer "Edge.Cuts") (width 0) (fill none))
+  (layer "F.Cu") (width 0) (fill solid))(gr_rect (start 10.508866497048132 60) (end 409.49113350295187 220) (layer "Edge.Cuts") (width 0) (fill none))
 )
