File: examples/aquila_gps.kicad_pcb (KiCad board)
At the start: 2 copper layers, 399 x 160 mm, 0 parts

Commit message: substrate sheet size is now set automatically
Other:
- board size 399 x 160 mm -> 399 x 149.4 mm
Changed lines of the file:
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@@
       (xy 308.9490823764759 199.203515625)
       (xy 308.9490823764759 190)
-      (xy 310.54205112647594 190)
-      (xy 310.54205112647594 190.451953125)
-      (xy 345.0893994446999 190.451953125)
-      (xy 345.0893994446999 189.203515625)
-      (xy 358.82186575221385 189.203515625)
-      (xy 358.82186575221385 180)
-      (xy 360.04159231471385 180)
-      (xy 360.04159231471385 144.596708005118)
-      (xy 397.26451274826604 144.596708005118)
-      (xy 397.26451274826604 80.58309195058654)
-      (xy 321.97218750616173 80.58309195058654)
-      (xy 321.97218750616173 144.596708005118)
-      (xy 359.1951079397139 144.596708005118)
-      (xy 359.1951079397139 180)
-      (xy 360.4148345022139 180)
-      (xy 360.4148345022139 189.10925688501632)
-      (xy 358.72760701223024 190.796484375)
-      (xy 345.0893994446999 190.796484375)
-      (xy 345.0893994446999 189.548046875)
-      (xy 274.401734058252 189.548046875)
-      (xy 274.401734058252 189.203515625)
-      (xy 260.66926775073796 189.203515625)
-      (xy 260.66926775073796 180)
-      (xy 260.29602556323795 180)
-      (xy 260.29602556323795 144.596708005118)
-      (xy 297.5189459967901 144.596708005118)
-      (xy 297.5189459967901 80.58309195058654)
-      (xy 222.22662075468583 80.58309195058654)
-      (xy 222.22662075468583 144.596708005118)
-      (xy 259.44954118823796 144.596708005118)
-      (xy 259.44954118823796 180)
-      (xy 259.07629900073795 180)
-      (xy 259.07629900073795 189.10925688501632)
-      (xy 260.76352649072163 190.796484375)
-      (xy 274.401734058252 190.796484375)
-      (xy 274.401734058252 190.451953125)
-      (xy 308.9490823764759 190.451953125)
-      (xy 308.9490823764759 190)
+      (xy 310.1688089389759 190)
+      (xy 310.1688089389759 154.596708005118)
+      (xy 347.39172937252806 154.596708005118)
+      (xy 347.39172937252806 90.58309195058654)
+      (xy 272.0994041304238 90.58309195058654)
+      (xy 272.0994041304238 154.596708005118)
+      (xy 309.32232456397594 154.596708005118)
+      (xy 309.32232456397594 190)
       (xy 310.54205112647594 190)
       (xy 310.54205112647594 199.10925688501632)
@@
       (xy 111.05091762352407 199.203515625)
       (xy 111.05091762352407 190)
-      (xy 111.05091762352407 190)
-      (xy 111.05091762352407 190.451953125)
-      (xy 145.59826594174802 190.451953125)
-      (xy 145.59826594174802 189.203515625)
-      (xy 159.33073224926204 189.203515625)
-      (xy 159.33073224926204 180)
-      (xy 160.55045881176204 180)
-      (xy 160.55045881176204 144.596708005118)
-      (xy 197.77337924531417 144.596708005118)
-      (xy 197.77337924531417 80.58309195058654)
-      (xy 122.48105400320989 80.58309195058654)
-      (xy 122.48105400320989 144.596708005118)
-      (xy 159.70397443676202 144.596708005118)
-      (xy 159.70397443676202 180)
-      (xy 160.92370099926202 180)
-      (xy 160.92370099926202 189.10925688501632)
-      (xy 159.23647350927837 190.796484375)
-      (xy 145.59826594174802 190.796484375)
-      (xy 145.59826594174802 189.548046875)
-      (xy 74.9106005553001 189.548046875)
-      (xy 74.9106005553001 189.203515625)
-      (xy 61.17813424778612 189.203515625)
-      (xy 61.17813424778612 180)
-      (xy 60.80489206028611 180)
-      (xy 60.80489206028611 144.596708005118)
-      (xy 98.02781249383824 144.596708005118)
-      (xy 98.02781249383824 80.58309195058654)
-      (xy 22.735487251733986 80.58309195058654)
-      (xy 22.735487251733986 144.596708005118)
-      (xy 59.95840768528612 144.596708005118)
-      (xy 59.95840768528612 180)
-      (xy 59.58516549778611 180)
-      (xy 59.58516549778611 189.10925688501632)
-      (xy 61.27239298776979 190.796484375)
-      (xy 74.9106005553001 190.796484375)
-      (xy 74.9106005553001 190.451953125)
-      (xy 109.45794887352406 190.451953125)
-      (xy 109.45794887352406 190)
+      (xy 110.67767543602406 190)
+      (xy 110.67767543602406 154.596708005118)
+      (xy 147.9005958695762 154.596708005118)
+      (xy 147.9005958695762 90.58309195058654)
+      (xy 72.60827062747194 90.58309195058654)
+      (xy 72.60827062747194 154.596708005118)
+      (xy 109.83119106102407 154.596708005118)
+      (xy 109.83119106102407 190)
       (xy 109.45794887352406 190)
       (xy 109.45794887352406 199.10925688501632)
@@
       (xy 210 200.451953125)
     )
-  (layer "F.Cu") (width 0) (fill solid))(gr_rect (start 10.508866497048132 60) (end 409.49113350295187 220) (layer "Edge.Cuts") (width 0) (fill none))
+  (layer "F.Cu") (width 0) (fill solid))(gr_rect (start 10.508866497048132 70.58309195058655) (end 409.49113350295187 220) (layer "Edge.Cuts") (width 0) (fill none))
 )

Commit message: fixed two-patch option bug
Other:
- board size 399 x 149.4 mm -> 399 x 159.4 mm
Changed lines of the file:
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@@
       (xy 308.9490823764759 199.203515625)
       (xy 308.9490823764759 190)
-      (xy 310.1688089389759 190)
-      (xy 310.1688089389759 154.596708005118)
-      (xy 347.39172937252806 154.596708005118)
-      (xy 347.39172937252806 90.58309195058654)
-      (xy 272.0994041304238 90.58309195058654)
-      (xy 272.0994041304238 154.596708005118)
-      (xy 309.32232456397594 154.596708005118)
-      (xy 309.32232456397594 190)
+      (xy 310.54205112647594 190)
+      (xy 310.54205112647594 190.451953125)
+      (xy 345.0893994446999 190.451953125)
+      (xy 345.0893994446999 189.203515625)
+      (xy 358.82186575221385 189.203515625)
+      (xy 358.82186575221385 180)
+      (xy 360.04159231471385 180)
+      (xy 360.04159231471385 144.596708005118)
+      (xy 397.26451274826604 144.596708005118)
+      (xy 397.26451274826604 80.58309195058654)
+      (xy 321.97218750616173 80.58309195058654)
+      (xy 321.97218750616173 144.596708005118)
+      (xy 359.1951079397139 144.596708005118)
+      (xy 359.1951079397139 180)
+      (xy 360.4148345022139 180)
+      (xy 360.4148345022139 189.10925688501632)
+      (xy 358.72760701223024 190.796484375)
+      (xy 345.0893994446999 190.796484375)
+      (xy 345.0893994446999 189.548046875)
+      (xy 274.401734058252 189.548046875)
+      (xy 274.401734058252 189.203515625)
+      (xy 260.66926775073796 189.203515625)
+      (xy 260.66926775073796 180)
+      (xy 260.29602556323795 180)
+      (xy 260.29602556323795 144.596708005118)
+      (xy 297.5189459967901 144.596708005118)
+      (xy 297.5189459967901 80.58309195058654)
+      (xy 222.22662075468583 80.58309195058654)
+      (xy 222.22662075468583 144.596708005118)
+      (xy 259.44954118823796 144.596708005118)
+      (xy 259.44954118823796 180)
+      (xy 259.07629900073795 180)
+      (xy 259.07629900073795 189.10925688501632)
+      (xy 260.76352649072163 190.796484375)
+      (xy 274.401734058252 190.796484375)
+      (xy 274.401734058252 190.451953125)
+      (xy 308.9490823764759 190.451953125)
+      (xy 308.9490823764759 190)
       (xy 310.54205112647594 190)
       (xy 310.54205112647594 199.10925688501632)
@@
       (xy 111.05091762352407 199.203515625)
       (xy 111.05091762352407 190)
-      (xy 110.67767543602406 190)
-      (xy 110.67767543602406 154.596708005118)
-      (xy 147.9005958695762 154.596708005118)
-      (xy 147.9005958695762 90.58309195058654)
-      (xy 72.60827062747194 90.58309195058654)
-      (xy 72.60827062747194 154.596708005118)
-      (xy 109.83119106102407 154.596708005118)
-      (xy 109.83119106102407 190)
+      (xy 111.05091762352407 190)
+      (xy 111.05091762352407 190.451953125)
+      (xy 145.59826594174802 190.451953125)
+      (xy 145.59826594174802 189.203515625)
+      (xy 159.33073224926204 189.203515625)
+      (xy 159.33073224926204 180)
+      (xy 160.55045881176204 180)
+      (xy 160.55045881176204 144.596708005118)
+      (xy 197.77337924531417 144.596708005118)
+      (xy 197.77337924531417 80.58309195058654)
+      (xy 122.48105400320989 80.58309195058654)
+      (xy 122.48105400320989 144.596708005118)
+      (xy 159.70397443676202 144.596708005118)
+      (xy 159.70397443676202 180)
+      (xy 160.92370099926202 180)
+      (xy 160.92370099926202 189.10925688501632)
+      (xy 159.23647350927837 190.796484375)
+      (xy 145.59826594174802 190.796484375)
+      (xy 145.59826594174802 189.548046875)
+      (xy 74.9106005553001 189.548046875)
+      (xy 74.9106005553001 189.203515625)
+      (xy 61.17813424778612 189.203515625)
+      (xy 61.17813424778612 180)
+      (xy 60.80489206028611 180)
+      (xy 60.80489206028611 144.596708005118)
+      (xy 98.02781249383824 144.596708005118)
+      (xy 98.02781249383824 80.58309195058654)
+      (xy 22.735487251733986 80.58309195058654)
+      (xy 22.735487251733986 144.596708005118)
+      (xy 59.95840768528612 144.596708005118)
+      (xy 59.95840768528612 180)
+      (xy 59.58516549778611 180)
+      (xy 59.58516549778611 189.10925688501632)
+      (xy 61.27239298776979 190.796484375)
+      (xy 74.9106005553001 190.796484375)
+      (xy 74.9106005553001 190.451953125)
+      (xy 109.45794887352406 190.451953125)
+      (xy 109.45794887352406 190)
       (xy 109.45794887352406 190)
       (xy 109.45794887352406 199.10925688501632)
@@
       (xy 210 200.451953125)
     )
-  (layer "F.Cu") (width 0) (fill solid))(gr_rect (start 10.508866497048132 70.58309195058655) (end 409.49113350295187 220) (layer "Edge.Cuts") (width 0) (fill none))
+  (layer "F.Cu") (width 0) (fill solid))(gr_rect (start 10.5 60.599999999999994) (end 409.5 220) (layer "Edge.Cuts") (width 0) (fill none))
 )

Commit message: implemented option for patch feed method
Other:
- board size 399 x 159.4 mm -> 399 x 134 mm
Changed lines of the file:
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@@
       (xy 245.34383269322396 199.203515625)
       (xy 308.9490823764759 199.203515625)
-      (xy 308.9490823764759 190)
-      (xy 310.54205112647594 190)
-      (xy 310.54205112647594 190.451953125)
-      (xy 345.0893994446999 190.451953125)
-      (xy 345.0893994446999 189.203515625)
-      (xy 358.82186575221385 189.203515625)
-      (xy 358.82186575221385 180)
-      (xy 360.04159231471385 180)
-      (xy 360.04159231471385 144.596708005118)
-      (xy 397.26451274826604 144.596708005118)
-      (xy 397.26451274826604 80.58309195058654)
-      (xy 321.97218750616173 80.58309195058654)
-      (xy 321.97218750616173 144.596708005118)
-      (xy 359.1951079397139 144.596708005118)
-      (xy 359.1951079397139 180)
-      (xy 360.4148345022139 180)
-      (xy 360.4148345022139 189.10925688501632)
-      (xy 358.72760701223024 190.796484375)
-      (xy 345.0893994446999 190.796484375)
-      (xy 345.0893994446999 189.548046875)
-      (xy 274.401734058252 189.548046875)
-      (xy 274.401734058252 189.203515625)
-      (xy 260.66926775073796 189.203515625)
-      (xy 260.66926775073796 180)
-      (xy 260.29602556323795 180)
-      (xy 260.29602556323795 144.596708005118)
-      (xy 297.5189459967901 144.596708005118)
-      (xy 297.5189459967901 80.58309195058654)
-      (xy 222.22662075468583 80.58309195058654)
-      (xy 222.22662075468583 144.596708005118)
-      (xy 259.44954118823796 144.596708005118)
-      (xy 259.44954118823796 180)
-      (xy 259.07629900073795 180)
-      (xy 259.07629900073795 189.10925688501632)
-      (xy 260.76352649072163 190.796484375)
-      (xy 274.401734058252 190.796484375)
-      (xy 274.401734058252 190.451953125)
-      (xy 308.9490823764759 190.451953125)
-      (xy 308.9490823764759 190)
-      (xy 310.54205112647594 190)
+      (xy 308.9490823764759 170)
+      (xy 310.54205112647594 170)
+      (xy 310.54205112647594 153.24110910190285)
+      (xy 311.3385355014759 153.24110910190285)
+      (xy 311.3385355014759 170)
+      (xy 347.39172937252806 170)
+      (xy 347.39172937252806 105.98638394546856)
+      (xy 272.0994041304238 105.98638394546856)
+      (xy 272.0994041304238 170)
+      (xy 308.15259800147595 170)
+      (xy 308.15259800147595 153.24110910190285)
+      (xy 308.9490823764759 153.24110910190285)
+      (xy 308.9490823764759 170)
+      (xy 310.54205112647594 170)
       (xy 310.54205112647594 199.10925688501632)
       (xy 308.85482363649226 200.796484375)
@@
       (xy 174.65616730677604 199.203515625)
       (xy 111.05091762352407 199.203515625)
-      (xy 111.05091762352407 190)
-      (xy 111.05091762352407 190)
-      (xy 111.05091762352407 190.451953125)
-      (xy 145.59826594174802 190.451953125)
-      (xy 145.59826594174802 189.203515625)
-      (xy 159.33073224926204 189.203515625)
-      (xy 159.33073224926204 180)
-      (xy 160.55045881176204 180)
-      (xy 160.55045881176204 144.596708005118)
-      (xy 197.77337924531417 144.596708005118)
-      (xy 197.77337924531417 80.58309195058654)
-      (xy 122.48105400320989 80.58309195058654)
-      (xy 122.48105400320989 144.596708005118)
-      (xy 159.70397443676202 144.596708005118)
-      (xy 159.70397443676202 180)
-      (xy 160.92370099926202 180)
-      (xy 160.92370099926202 189.10925688501632)
-      (xy 159.23647350927837 190.796484375)
-      (xy 145.59826594174802 190.796484375)
-      (xy 145.59826594174802 189.548046875)
-      (xy 74.9106005553001 189.548046875)
-      (xy 74.9106005553001 189.203515625)
-      (xy 61.17813424778612 189.203515625)
-      (xy 61.17813424778612 180)
-      (xy 60.80489206028611 180)
-      (xy 60.80489206028611 144.596708005118)
-      (xy 98.02781249383824 144.596708005118)
-      (xy 98.02781249383824 80.58309195058654)
-      (xy 22.735487251733986 80.58309195058654)
-      (xy 22.735487251733986 144.596708005118)
-      (xy 59.95840768528612 144.596708005118)
-      (xy 59.95840768528612 180)
-      (xy 59.58516549778611 180)
-      (xy 59.58516549778611 189.10925688501632)
-      (xy 61.27239298776979 190.796484375)
-      (xy 74.9106005553001 190.796484375)
-      (xy 74.9106005553001 190.451953125)
-      (xy 109.45794887352406 190.451953125)
-      (xy 109.45794887352406 190)
-      (xy 109.45794887352406 190)
+      (xy 111.05091762352407 170)
+      (xy 111.05091762352407 170)
+      (xy 111.05091762352407 153.24110910190285)
+      (xy 111.84740199852406 153.24110910190285)
+      (xy 111.84740199852406 170)
+      (xy 147.9005958695762 170)
+      (xy 147.9005958695762 105.98638394546856)
+      (xy 72.60827062747194 105.98638394546856)
+      (xy 72.60827062747194 170)
+      (xy 108.66146449852407 170)
+      (xy 108.66146449852407 153.24110910190285)
+      (xy 109.45794887352406 153.24110910190285)
+      (xy 109.45794887352406 170)
+      (xy 109.45794887352406 170)
       (xy 109.45794887352406 199.10925688501632)
       (xy 111.14517636350774 200.796484375)
@@
       (xy 210 200.451953125)
     )
-  (layer "F.Cu") (width 0) (fill solid))(gr_rect (start 10.5 60.599999999999994) (end 409.5 220) (layer "Edge.Cuts") (width 0) (fill none))
+  (layer "F.Cu") (width 0) (fill solid))(gr_rect (start 10.5 86.0) (end 409.5 220) (layer "Edge.Cuts") (width 0) (fill none))
 )

Commit message: implemented square patches with trimmed corners for circular polarisation
Other:
- board size 399 x 134 mm -> 399 x 159.4 mm
Changed lines of the file:
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@@
       (xy 245.34383269322396 199.203515625)
       (xy 308.9490823764759 199.203515625)
-      (xy 308.9490823764759 170)
-      (xy 310.54205112647594 170)
-      (xy 310.54205112647594 153.24110910190285)
-      (xy 311.3385355014759 153.24110910190285)
-      (xy 311.3385355014759 170)
-      (xy 347.39172937252806 170)
-      (xy 347.39172937252806 105.98638394546856)
-      (xy 272.0994041304238 105.98638394546856)
-      (xy 272.0994041304238 170)
-      (xy 308.15259800147595 170)
-      (xy 308.15259800147595 153.24110910190285)
-      (xy 308.9490823764759 153.24110910190285)
-      (xy 308.9490823764759 170)
-      (xy 310.54205112647594 170)
+      (xy 308.9490823764759 190)
+      (xy 310.54205112647594 190)
+      (xy 310.54205112647594 190.451953125)
+      (xy 345.0893994446999 190.451953125)
+      (xy 345.0893994446999 189.203515625)
+      (xy 358.82186575221385 189.203515625)
+      (xy 358.82186575221385 180)
+      (xy 360.04159231471385 180)
+      (xy 360.04159231471385 144.596708005118)
+      (xy 397.26451274826604 144.596708005118)
+      (xy 397.26451274826604 80.58309195058654)
+      (xy 321.97218750616173 80.58309195058654)
+      (xy 321.97218750616173 144.596708005118)
+      (xy 359.1951079397139 144.596708005118)
+      (xy 359.1951079397139 180)
+      (xy 360.4148345022139 180)
+      (xy 360.4148345022139 189.10925688501632)
+      (xy 358.72760701223024 190.796484375)
+      (xy 345.0893994446999 190.796484375)
+      (xy 345.0893994446999 189.548046875)
+      (xy 274.401734058252 189.548046875)
+      (xy 274.401734058252 189.203515625)
+      (xy 260.66926775073796 189.203515625)
+      (xy 260.66926775073796 180)
+      (xy 260.29602556323795 180)
+      (xy 260.29602556323795 144.596708005118)
+      (xy 297.5189459967901 144.596708005118)
+      (xy 297.5189459967901 80.58309195058654)
+      (xy 222.22662075468583 80.58309195058654)
+      (xy 222.22662075468583 144.596708005118)
+      (xy 259.44954118823796 144.596708005118)
+      (xy 259.44954118823796 180)
+      (xy 259.07629900073795 180)
+      (xy 259.07629900073795 189.10925688501632)
+      (xy 260.76352649072163 190.796484375)
+      (xy 274.401734058252 190.796484375)
+      (xy 274.401734058252 190.451953125)
+      (xy 308.9490823764759 190.451953125)
+      (xy 308.9490823764759 190)
+      (xy 310.54205112647594 190)
       (xy 310.54205112647594 199.10925688501632)
       (xy 308.85482363649226 200.796484375)
@@
       (xy 174.65616730677604 199.203515625)
       (xy 111.05091762352407 199.203515625)
-      (xy 111.05091762352407 170)
-      (xy 111.05091762352407 170)
-      (xy 111.05091762352407 153.24110910190285)
-      (xy 111.84740199852406 153.24110910190285)
-      (xy 111.84740199852406 170)
-      (xy 147.9005958695762 170)
-      (xy 147.9005958695762 105.98638394546856)
-      (xy 72.60827062747194 105.98638394546856)
-      (xy 72.60827062747194 170)
-      (xy 108.66146449852407 170)
-      (xy 108.66146449852407 153.24110910190285)
-      (xy 109.45794887352406 153.24110910190285)
-      (xy 109.45794887352406 170)
-      (xy 109.45794887352406 170)
+      (xy 111.05091762352407 190)
+      (xy 111.05091762352407 190)
+      (xy 111.05091762352407 190.451953125)
+      (xy 145.59826594174802 190.451953125)
+      (xy 145.59826594174802 189.203515625)
+      (xy 159.33073224926204 189.203515625)
+      (xy 159.33073224926204 180)
+      (xy 160.55045881176204 180)
+      (xy 160.55045881176204 144.596708005118)
+      (xy 197.77337924531417 144.596708005118)
+      (xy 197.77337924531417 80.58309195058654)
+      (xy 122.48105400320989 80.58309195058654)
+      (xy 122.48105400320989 144.596708005118)
+      (xy 159.70397443676202 144.596708005118)
+      (xy 159.70397443676202 180)
+      (xy 160.92370099926202 180)
+      (xy 160.92370099926202 189.10925688501632)
+      (xy 159.23647350927837 190.796484375)
+      (xy 145.59826594174802 190.796484375)
+      (xy 145.59826594174802 189.548046875)
+      (xy 74.9106005553001 189.548046875)
+      (xy 74.9106005553001 189.203515625)
+      (xy 61.17813424778612 189.203515625)
+      (xy 61.17813424778612 180)
+      (xy 60.80489206028611 180)
+      (xy 60.80489206028611 144.596708005118)
+      (xy 98.02781249383824 144.596708005118)
+      (xy 98.02781249383824 80.58309195058654)
+      (xy 22.735487251733986 80.58309195058654)
+      (xy 22.735487251733986 144.596708005118)
+      (xy 59.95840768528612 144.596708005118)
+      (xy 59.95840768528612 180)
+      (xy 59.58516549778611 180)
+      (xy 59.58516549778611 189.10925688501632)
+      (xy 61.27239298776979 190.796484375)
+      (xy 74.9106005553001 190.796484375)
+      (xy 74.9106005553001 190.451953125)
+      (xy 109.45794887352406 190.451953125)
+      (xy 109.45794887352406 190)
+      (xy 109.45794887352406 190)
       (xy 109.45794887352406 199.10925688501632)
       (xy 111.14517636350774 200.796484375)
@@
       (xy 210 200.451953125)
     )
-  (layer "F.Cu") (width 0) (fill solid))(gr_rect (start 10.5 86.0) (end 409.5 220) (layer "Edge.Cuts") (width 0) (fill none))
+  (layer "F.Cu") (width 0) (fill solid))(gr_rect (start 10.5 60.599999999999994) (end 409.5 220) (layer "Edge.Cuts") (width 0) (fill none))
 )
