File: examples/aquila_gps.kicad_pcb (KiCad board)
At the start: 2 copper layers, 399 x 159.4 mm, 0 parts

Commit message: removed nested IFs for array assembly
Other:
- board size 399 x 159.4 mm -> 399 x 159.6 mm
Changed lines of the file:
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@@
       (xy 358.82186575221385 189.203515625)
       (xy 358.82186575221385 180)
-      (xy 360.04159231471385 180)
-      (xy 360.04159231471385 144.596708005118)
-      (xy 397.26451274826604 144.596708005118)
-      (xy 397.26451274826604 80.58309195058654)
-      (xy 321.97218750616173 80.58309195058654)
-      (xy 321.97218750616173 144.596708005118)
-      (xy 359.1951079397139 144.596708005118)
-      (xy 359.1951079397139 180)
+      (xy 359.9841704397139 180)
+      (xy 359.9841704397139 144.4680102788262)
+      (xy 391.6532391150921 144.4680102788262)
+      (xy 391.6532391150921 88.40695455003927)
+      (xy 383.64451686812254 80.3982323030697)
+      (xy 327.58346113933567 80.3982323030697)
+      (xy 327.58346113933567 136.45928803185663)
+      (xy 335.59218338630524 144.4680102788262)
+      (xy 359.25252981471385 144.4680102788262)
+      (xy 359.25252981471385 180)
       (xy 360.4148345022139 180)
       (xy 360.4148345022139 189.10925688501632)
@@
       (xy 260.66926775073796 189.203515625)
       (xy 260.66926775073796 180)
-      (xy 260.29602556323795 180)
-      (xy 260.29602556323795 144.596708005118)
-      (xy 297.5189459967901 144.596708005118)
-      (xy 297.5189459967901 80.58309195058654)
-      (xy 222.22662075468583 80.58309195058654)
-      (xy 222.22662075468583 144.596708005118)
-      (xy 259.44954118823796 144.596708005118)
-      (xy 259.44954118823796 180)
+      (xy 260.23860368823796 180)
+      (xy 260.23860368823796 144.4680102788262)
+      (xy 291.9076723636162 144.4680102788262)
+      (xy 291.9076723636162 88.40695455003927)
+      (xy 283.89895011664663 80.3982323030697)
+      (xy 227.83789438785973 80.3982323030697)
+      (xy 227.83789438785973 136.45928803185663)
+      (xy 235.84661663482927 144.4680102788262)
+      (xy 259.50696306323795 144.4680102788262)
+      (xy 259.50696306323795 180)
       (xy 259.07629900073795 180)
       (xy 259.07629900073795 189.10925688501632)
@@
       (xy 159.33073224926204 189.203515625)
       (xy 159.33073224926204 180)
-      (xy 160.55045881176204 180)
-      (xy 160.55045881176204 144.596708005118)
-      (xy 197.77337924531417 144.596708005118)
-      (xy 197.77337924531417 80.58309195058654)
-      (xy 122.48105400320989 80.58309195058654)
-      (xy 122.48105400320989 144.596708005118)
-      (xy 159.70397443676202 144.596708005118)
-      (xy 159.70397443676202 180)
+      (xy 160.49303693676202 180)
+      (xy 160.49303693676202 144.4680102788262)
+      (xy 192.16210561214027 144.4680102788262)
+      (xy 192.16210561214027 88.40695455003927)
+      (xy 184.15338336517073 80.3982323030697)
+      (xy 128.0923276363838 80.3982323030697)
+      (xy 128.0923276363838 136.45928803185663)
+      (xy 136.10104988335337 144.4680102788262)
+      (xy 159.76139631176204 144.4680102788262)
+      (xy 159.76139631176204 180)
       (xy 160.92370099926202 180)
       (xy 160.92370099926202 189.10925688501632)
@@
       (xy 61.17813424778612 189.203515625)
       (xy 61.17813424778612 180)
-      (xy 60.80489206028611 180)
-      (xy 60.80489206028611 144.596708005118)
-      (xy 98.02781249383824 144.596708005118)
-      (xy 98.02781249383824 80.58309195058654)
-      (xy 22.735487251733986 80.58309195058654)
-      (xy 22.735487251733986 144.596708005118)
-      (xy 59.95840768528612 144.596708005118)
-      (xy 59.95840768528612 180)
+      (xy 60.74747018528612 180)
+      (xy 60.74747018528612 144.4680102788262)
+      (xy 92.41653886066436 144.4680102788262)
+      (xy 92.41653886066436 88.40695455003927)
+      (xy 84.40781661369479 80.3982323030697)
+      (xy 28.346760884907866 80.3982323030697)
+      (xy 28.346760884907866 136.45928803185663)
+      (xy 36.355483131877435 144.4680102788262)
+      (xy 60.01582956028611 144.4680102788262)
+      (xy 60.01582956028611 180)
       (xy 59.58516549778611 180)
       (xy 59.58516549778611 189.10925688501632)
@@
       (xy 210 200.451953125)
     )
-  (layer "F.Cu") (width 0) (fill solid))(gr_rect (start 10.5 60.599999999999994) (end 409.5 220) (layer "Edge.Cuts") (width 0) (fill none))
+  (layer "F.Cu") (width 0) (fill solid))(gr_rect (start 10.5 60.400000000000006) (end 409.5 220) (layer "Edge.Cuts") (width 0) (fill none))
 )
