File: examples/aquila_telem.kicad_pcb (KiCad board)
At the start: 2 copper layers, 399 x 160 mm, 0 parts

Commit message: substrate sheet size is now set automatically
Other:
- board size 399 x 160 mm -> 399 x 221.3 mm
Changed lines of the file:
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@@
       (xy 210 200.451953125)
     )
-  (layer "F.Cu") (width 0) (fill solid))(gr_rect (start 10.508866497048132 60) (end 409.49113350295187 220) (layer "Edge.Cuts") (width 0) (fill none))
+  (layer "F.Cu") (width 0) (fill solid))(gr_rect (start 10.508866497048132 -1.2731006311007604) (end 409.49113350295187 220) (layer "Edge.Cuts") (width 0) (fill none))
 )

Commit message: fixed two-patch option bug
Changed lines of the file:
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@@
       (xy 210 200.451953125)
     )
-  (layer "F.Cu") (width 0) (fill solid))(gr_rect (start 10.508866497048132 -1.2731006311007604) (end 409.49113350295187 220) (layer "Edge.Cuts") (width 0) (fill none))
+  (layer "F.Cu") (width 0) (fill solid))(gr_rect (start 10.5 -1.2700000000000102) (end 409.5 220) (layer "Edge.Cuts") (width 0) (fill none))
 )

Commit message: implemented option for patch feed method
Other:
- board size 399 x 221.3 mm -> 399 x 186.3 mm
Changed lines of the file:
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@@
     (gr_poly
     (pts
-      (xy 270.83774479981173 200.451953125)
-      (xy 270.83774479981173 199.203515625)
+      (xy 274.13195448367253 200.451953125)
+      (xy 274.13195448367253 199.203515625)
       (xy 308.9490823764759 199.203515625)
-      (xy 308.9490823764759 190)
-      (xy 310.1688089389759 190)
-      (xy 310.1688089389759 129.0599072219244)
-      (xy 374.5463384762378 129.0599072219244)
-      (xy 374.5463384762378 18.72689936889924)
-      (xy 244.94479502671408 18.72689936889924)
-      (xy 244.94479502671408 129.0599072219244)
-      (xy 309.32232456397594 129.0599072219244)
-      (xy 309.32232456397594 190)
-      (xy 310.54205112647594 190)
+      (xy 308.9490823764759 170)
+      (xy 310.54205112647594 170)
+      (xy 310.54205112647594 139.54773109950514)
+      (xy 311.3385355014759 139.54773109950514)
+      (xy 311.3385355014759 170)
+      (xy 378.0551360235463 170)
+      (xy 378.0551360235463 53.68204905451327)
+      (xy 241.43599747940553 53.68204905451327)
+      (xy 241.43599747940553 170)
+      (xy 308.15259800147595 170)
+      (xy 308.15259800147595 139.54773109950514)
+      (xy 308.9490823764759 139.54773109950514)
+      (xy 308.9490823764759 170)
+      (xy 310.54205112647594 170)
       (xy 310.54205112647594 199.10925688501632)
       (xy 308.85482363649226 200.796484375)
-      (xy 270.83774479981173 200.796484375)
-      (xy 270.83774479981173 199.548046875)
-      (xy 149.16225520018827 199.548046875)
-      (xy 149.16225520018827 199.203515625)
+      (xy 274.13195448367253 200.796484375)
+      (xy 274.13195448367253 199.548046875)
+      (xy 145.8680455163275 199.548046875)
+      (xy 145.8680455163275 199.203515625)
       (xy 111.05091762352407 199.203515625)
-      (xy 111.05091762352407 190)
-      (xy 110.67767543602406 190)
-      (xy 110.67767543602406 129.0599072219244)
-      (xy 175.05520497328592 129.0599072219244)
-      (xy 175.05520497328592 18.72689936889924)
-      (xy 45.45366152376221 18.72689936889924)
-      (xy 45.45366152376221 129.0599072219244)
-      (xy 109.83119106102407 129.0599072219244)
-      (xy 109.83119106102407 190)
-      (xy 109.45794887352406 190)
+      (xy 111.05091762352407 170)
+      (xy 111.05091762352407 170)
+      (xy 111.05091762352407 139.54773109950514)
+      (xy 111.84740199852406 139.54773109950514)
+      (xy 111.84740199852406 170)
+      (xy 178.56400252059447 170)
+      (xy 178.56400252059447 53.68204905451327)
+      (xy 41.94486397645366 53.68204905451327)
+      (xy 41.94486397645366 170)
+      (xy 108.66146449852407 170)
+      (xy 108.66146449852407 139.54773109950514)
+      (xy 109.45794887352406 139.54773109950514)
+      (xy 109.45794887352406 170)
+      (xy 109.45794887352406 170)
       (xy 109.45794887352406 199.10925688501632)
       (xy 111.14517636350774 200.796484375)
-      (xy 149.16225520018827 200.796484375)
-      (xy 149.16225520018827 200.451953125)
+      (xy 145.8680455163275 200.796484375)
+      (xy 145.8680455163275 200.451953125)
       (xy 210 200.451953125)
       (xy 210 200.3)
@@
       (xy 210 200.451953125)
     )
-  (layer "F.Cu") (width 0) (fill solid))(gr_rect (start 10.5 -1.2700000000000102) (end 409.5 220) (layer "Edge.Cuts") (width 0) (fill none))
+  (layer "F.Cu") (width 0) (fill solid))(gr_rect (start 10.5 33.69999999999999) (end 409.5 220) (layer "Edge.Cuts") (width 0) (fill none))
 )
