File: examples/aquila_telem.kicad_pcb (KiCad board)
At the start: 2 copper layers, 399 x 186.3 mm, 0 parts

Commit message: removed nested IFs for array assembly
Other:
- board size 399 x 186.3 mm -> 399 x 166.3 mm
Changed lines of the file:
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@@
       (xy 274.13195448367253 199.203515625)
       (xy 308.9490823764759 199.203515625)
-      (xy 308.9490823764759 170)
-      (xy 310.54205112647594 170)
-      (xy 310.54205112647594 139.54773109950514)
-      (xy 312.13501987647595 139.54773109950514)
-      (xy 312.13501987647595 170)
-      (xy 378.0551360235463 170)
-      (xy 378.0551360235463 53.68204905451327)
-      (xy 241.43599747940553 53.68204905451327)
-      (xy 241.43599747940553 170)
-      (xy 307.3561136264759 170)
-      (xy 307.3561136264759 139.54773109950514)
-      (xy 308.9490823764759 139.54773109950514)
-      (xy 308.9490823764759 170)
-      (xy 310.54205112647594 170)
+      (xy 308.9490823764759 190)
+      (xy 310.54205112647594 190)
+      (xy 310.54205112647594 159.54773109950514)
+      (xy 312.13501987647595 159.54773109950514)
+      (xy 312.13501987647595 190)
+      (xy 378.0551360235463 190)
+      (xy 378.0551360235463 73.68204905451327)
+      (xy 241.43599747940553 73.68204905451327)
+      (xy 241.43599747940553 190)
+      (xy 307.3561136264759 190)
+      (xy 307.3561136264759 159.54773109950514)
+      (xy 308.9490823764759 159.54773109950514)
+      (xy 308.9490823764759 190)
+      (xy 310.54205112647594 190)
       (xy 310.54205112647594 199.10925688501632)
       (xy 308.85482363649226 200.796484375)
@@
       (xy 145.8680455163275 199.203515625)
       (xy 111.05091762352407 199.203515625)
-      (xy 111.05091762352407 170)
-      (xy 111.05091762352407 170)
-      (xy 111.05091762352407 139.54773109950514)
-      (xy 112.64388637352407 139.54773109950514)
-      (xy 112.64388637352407 170)
-      (xy 178.56400252059447 170)
-      (xy 178.56400252059447 53.68204905451327)
-      (xy 41.94486397645366 53.68204905451327)
-      (xy 41.94486397645366 170)
-      (xy 107.86498012352406 170)
-      (xy 107.86498012352406 139.54773109950514)
-      (xy 109.45794887352406 139.54773109950514)
-      (xy 109.45794887352406 170)
-      (xy 109.45794887352406 170)
+      (xy 111.05091762352407 190)
+      (xy 111.05091762352407 190)
+      (xy 111.05091762352407 159.54773109950514)
+      (xy 112.64388637352407 159.54773109950514)
+      (xy 112.64388637352407 190)
+      (xy 178.56400252059447 190)
+      (xy 178.56400252059447 73.68204905451327)
+      (xy 41.94486397645366 73.68204905451327)
+      (xy 41.94486397645366 190)
+      (xy 107.86498012352406 190)
+      (xy 107.86498012352406 159.54773109950514)
+      (xy 109.45794887352406 159.54773109950514)
+      (xy 109.45794887352406 190)
+      (xy 109.45794887352406 190)
       (xy 109.45794887352406 199.10925688501632)
       (xy 111.14517636350774 200.796484375)
@@
       (xy 210 200.451953125)
     )
-  (layer "F.Cu") (width 0) (fill solid))(gr_rect (start 10.5 33.69999999999999) (end 409.5 220) (layer "Edge.Cuts") (width 0) (fill none))
+  (layer "F.Cu") (width 0) (fill solid))(gr_rect (start 10.5 53.69999999999999) (end 409.5 220) (layer "Edge.Cuts") (width 0) (fill none))
 )
