File: examples/aquila_gps2.kicad_pcb (KiCad board)
At the start: 2 copper layers, 399 x 186.3 mm, 0 parts

Commit message: implemented square patches with trimmed corners for circular polarisation
Other:
- board size 399 x 186.3 mm -> 399 x 149.5 mm
Changed lines of the file:
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@@
     (gr_poly
     (pts
-      (xy 274.13195448367253 200.451953125)
-      (xy 274.13195448367253 199.203515625)
+      (xy 245.34383269322396 200.451953125)
+      (xy 245.34383269322396 199.203515625)
       (xy 308.9490823764759 199.203515625)
-      (xy 308.9490823764759 170)
-      (xy 310.54205112647594 170)
-      (xy 310.54205112647594 139.54773109950514)
-      (xy 312.13501987647595 139.54773109950514)
-      (xy 312.13501987647595 170)
-      (xy 378.0551360235463 170)
-      (xy 378.0551360235463 53.68204905451327)
-      (xy 241.43599747940553 53.68204905451327)
-      (xy 241.43599747940553 170)
-      (xy 307.3561136264759 170)
-      (xy 307.3561136264759 139.54773109950514)
-      (xy 308.9490823764759 139.54773109950514)
-      (xy 308.9490823764759 170)
-      (xy 310.54205112647594 170)
+      (xy 308.9490823764759 190)
+      (xy 310.1688089389759 190)
+      (xy 310.1688089389759 154.596708005118)
+      (xy 341.7804557393542 154.596708005118)
+      (xy 341.7804557393542 98.53565227633106)
+      (xy 333.7717334923846 90.5269300293615)
+      (xy 277.7106777635977 90.5269300293615)
+      (xy 277.7106777635977 146.58798575814842)
+      (xy 285.71940001056726 154.596708005118)
+      (xy 309.32232456397594 154.596708005118)
+      (xy 309.32232456397594 190)
+      (xy 310.54205112647594 190)
       (xy 310.54205112647594 199.10925688501632)
       (xy 308.85482363649226 200.796484375)
-      (xy 274.13195448367253 200.796484375)
-      (xy 274.13195448367253 199.548046875)
-      (xy 145.8680455163275 199.548046875)
-      (xy 145.8680455163275 199.203515625)
+      (xy 245.34383269322396 200.796484375)
+      (xy 245.34383269322396 199.548046875)
+      (xy 174.65616730677604 199.548046875)
+      (xy 174.65616730677604 199.203515625)
       (xy 111.05091762352407 199.203515625)
-      (xy 111.05091762352407 170)
-      (xy 111.05091762352407 170)
-      (xy 111.05091762352407 139.54773109950514)
-      (xy 112.64388637352407 139.54773109950514)
-      (xy 112.64388637352407 170)
-      (xy 178.56400252059447 170)
-      (xy 178.56400252059447 53.68204905451327)
-      (xy 41.94486397645366 53.68204905451327)
-      (xy 41.94486397645366 170)
-      (xy 107.86498012352406 170)
-      (xy 107.86498012352406 139.54773109950514)
-      (xy 109.45794887352406 139.54773109950514)
-      (xy 109.45794887352406 170)
-      (xy 109.45794887352406 170)
+      (xy 111.05091762352407 190)
+      (xy 110.67767543602406 190)
+      (xy 110.67767543602406 154.596708005118)
+      (xy 142.2893222364023 154.596708005118)
+      (xy 142.2893222364023 98.53565227633106)
+      (xy 134.28059998943274 90.5269300293615)
+      (xy 78.21954426064582 90.5269300293615)
+      (xy 78.21954426064582 146.58798575814842)
+      (xy 86.22826650761539 154.596708005118)
+      (xy 109.83119106102407 154.596708005118)
+      (xy 109.83119106102407 190)
+      (xy 109.45794887352406 190)
       (xy 109.45794887352406 199.10925688501632)
       (xy 111.14517636350774 200.796484375)
-      (xy 145.8680455163275 200.796484375)
-      (xy 145.8680455163275 200.451953125)
+      (xy 174.65616730677604 200.796484375)
+      (xy 174.65616730677604 200.451953125)
       (xy 210 200.451953125)
       (xy 210 200.3)
@@
       (xy 210 200.451953125)
     )
-  (layer "F.Cu") (width 0) (fill solid))(gr_rect (start 10.5 33.69999999999999) (end 409.5 220) (layer "Edge.Cuts") (width 0) (fill none))
+  (layer "F.Cu") (width 0) (fill solid))(gr_rect (start 10.5 70.5) (end 409.5 220) (layer "Edge.Cuts") (width 0) (fill none))
 )
